File: Diff_amp.kicad_pcb (KiCad board)
At the start: 2 copper layers, 15 parts, among them J1 Conn_01x01, J10 Conn_01x01, J2 Conn_01x01, J3 Conn_01x01, J4 Conn_01x01, J5 Conn_01x01, J6 Conn_01x01, J7 Conn_01x01, J8 Conn_01x01, J9 Conn_01x01, Q1 IRF540N, Q2 IRF540N

Commit message: Placements done
Parts:
- moved J9 39.4 mm to (65.7, 78.5)
- moved J10 25.4 mm to (81.1, 78.5)
- moved J7 22.1 mm to (96.6, 78.5)
- moved R3 21.1 mm to (90.6, 57.6)
- moved J5 19.9 mm to (71.5, 57.5)
- moved J1 19.2 mm to (50.2, 57.5)
- moved J8 16.9 mm to (96.5, 31.6)
- moved Q2 13.8 mm to (79.9, 67.6)
- moved J4 10.9 mm to (81.1, 31.6)
- moved Q1 9.38 mm to (57.1, 67.6)
- moved R1 9.35 mm to (59.5, 42.4)
- moved R2 8.40 mm to (67.2, 42.4), turned to 0 degrees
- moved J6 5.79 mm to (65.6, 31.6)
- moved J2 4.53 mm to (50.2, 78.5)
Changed lines of the file:
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@@
 	(footprint "Connector_PinHeader_2.54mm:PinHeader_1x01_P2.54mm_Vertical"
 		(layer "F.Cu")
-		(at 47.07 76.46 90)
+		(at 50.22 57.5 90)
 		(descr "Through hole straight pin header, 1x01, 2.54mm pitch, single row")
 		(tags "Through hole pin header THT 1x01 2.54mm single row")
 		(property "Reference" "J1"
-			(at 0 -2.38 90)
+			(at 2.68 -0.15 180)
 			(layer "F.SilkS")
 			(effects
@@
 	(footprint "Connector_PinHeader_2.54mm:PinHeader_1x01_P2.54mm_Vertical"
 		(layer "F.Cu")
-		(at 65.64 76.48 -90)
+		(at 71.48 57.5 -90)
 		(descr "Through hole straight pin header, 1x01, 2.54mm pitch, single row")
 		(tags "Through hole pin header THT 1x01 2.54mm single row")
 		(property "Reference" "J5"
-			(at 0 -2.38 90)
+			(at -2.84 -0.05 180)
 			(layer "F.SilkS")
 			(effects
@@
 	(footprint "Resistor_THT:R_Axial_DIN0309_L9.0mm_D3.2mm_P15.24mm_Horizontal"
 		(layer "F.Cu")
-		(at 58.85 41.9 -90)
+		(at 67.24 42.37)
 		(descr "Resistor, Axial_DIN0309 series, Axial, Horizontal, pin pitch=15.24mm, 0.5W = 1/2W, length*diameter=9*3.2mm^2, http://cdn-reichelt.de/documents/datenblatt/B400/1_4W%23YAG.pdf")
 		(tags "Resistor Axial_DIN0309 series Axial Horizontal pin pitch 15.24mm 0.5W = 1/2W length 9mm diameter 3.2mm")
 		(property "Reference" "R2"
-			(at 7.62 -2.72 90)
+			(at 7.95 -3.17 180)
 			(layer "F.SilkS")
 			(effects
@@
 		)
 		(property "Value" "R"
-			(at 7.62 2.72 90)
+			(at 7.62 2.72 0)
 			(layer "F.Fab")
 			(effects
@@
 		)
 		(property "Datasheet" ""
-			(at 0 0 90)
+			(at 0 0 0)
 			(layer "F.Fab")
 			(hide yes)
@@
 		)
 		(property "Description" "Resistor"
-			(at 0 0 90)
+			(at 0 0 0)
 			(layer "F.Fab")
 			(hide yes)
@@
 		)
 		(property "KiLib_Generator" "resistor/THT"
-			(at 0 0 90)
+			(at 0 0 0)
 			(layer "F.SilkS")
 			(hide yes)
@@
 		)
 		(fp_text user "${REFERENCE}"
-			(at 7.62 0 90)
+			(at 7.62 0 0)
 			(layer "F.Fab")
 			(effects
@@
 		)
 		(pad "1" thru_hole circle
-			(at 0 0 270)
+			(at 0 0)
 			(size 1.6 1.6)
 			(drill 0.8)
@@
 		)
 		(pad "2" thru_hole circle
-			(at 15.24 0 270)
+			(at 15.24 0)
 			(size 1.6 1.6)
 			(drill 0.8)
@@
 	(footprint "Connector_PinHeader_2.54mm:PinHeader_1x01_P2.54mm_Vertical"
 		(layer "F.Cu")
-		(at 85.39 53.44)
+		(at 81.126 78.5)
 		(descr "Through hole straight pin header, 1x01, 2.54mm pitch, single row")
 		(tags "Through hole pin header THT 1x01 2.54mm single row")
@@
 	(footprint "Connector_PinHeader_2.54mm:PinHeader_1x01_P2.54mm_Vertical"
 		(layer "F.Cu")
-		(at 74.61 76.43 -90)
+		(at 96.579 78.5 -90)
 		(descr "Through hole straight pin header, 1x01, 2.54mm pitch, single row")
 		(tags "Through hole pin header THT 1x01 2.54mm single row")
 		(property "Reference" "J7"
-			(at 0 -2.38 90)
+			(at -2.8 -0.071 180)
 			(layer "F.SilkS")
 			(effects
@@
 	(footprint "Resistor_THT:R_Axial_DIN0309_L9.0mm_D3.2mm_P15.24mm_Horizontal"
 		(layer "F.Cu")
-		(at 50.14 41.9 -90)
+		(at 59.48 42.37 -90)
 		(descr "Resistor, Axial_DIN0309 series, Axial, Horizontal, pin pitch=15.24mm, 0.5W = 1/2W, length*diameter=9*3.2mm^2, http://cdn-reichelt.de/documents/datenblatt/B400/1_4W%23YAG.pdf")
 		(tags "Resistor Axial_DIN0309 series Axial Horizontal pin pitch 15.24mm 0.5W = 1/2W length 9mm diameter 3.2mm")
 		(property "Reference" "R1"
-			(at 7.62 -2.72 90)
+			(at -1.95 -0.03 180)
 			(layer "F.SilkS")
 			(effects
@@
 	(footprint "Package_TO_SOT_THT:TO-220-3_Vertical"
 		(layer "F.Cu")
-		(at 47.73 68.29)
+		(at 57.08 67.59)
 		(descr "TO-220-3, Vertical, RM 2.54mm, see https://www.vishay.com/docs/66542/to-220-1.pdf")
 		(tags "TO-220-3 Vertical RM 2.54mm")
@@
 	(footprint "Connector_PinHeader_2.54mm:PinHeader_1x01_P2.54mm_Vertical"
 		(layer "F.Cu")
-		(at 54.26 76.46 90)
+		(at 50.22 78.5 90)
 		(descr "Through hole straight pin header, 1x01, 2.54mm pitch, single row")
 		(tags "Through hole pin header THT 1x01 2.54mm single row")
 		(property "Reference" "J2"
-			(at 0 -2.38 90)
+			(at 2.74 0.12 180)
 			(layer "F.SilkS")
 			(effects
@@
 	)
 	(footprint "Connector_PinHeader_2.54mm:PinHeader_1x01_P2.54mm_Vertical"
+		(locked yes)
 		(layer "F.Cu")
-		(at 70.15 31.77)
+		(at 81.066667 31.62)
 		(descr "Through hole straight pin header, 1x01, 2.54mm pitch, single row")
 		(tags "Through hole pin header THT 1x01 2.54mm single row")
@@
 	(footprint "Package_TO_SOT_THT:TO-220-3_Vertical"
 		(layer "F.Cu")
-		(at 66.17 68.62)
+		(at 79.94 67.59)
 		(descr "TO-220-3, Vertical, RM 2.54mm, see https://www.vishay.com/docs/66542/to-220-1.pdf")
 		(tags "TO-220-3 Vertical RM 2.54mm")
@@
 	(footprint "Connector_PinHeader_2.54mm:PinHeader_1x01_P2.54mm_Vertical"
 		(layer "F.Cu")
-		(at 85.32 44.32)
+		(at 65.673 78.5)
 		(descr "Through hole straight pin header, 1x01, 2.54mm pitch, single row")
 		(tags "Through hole pin header THT 1x01 2.54mm single row")
@@
 	)
 	(footprint "Connector_PinHeader_2.54mm:PinHeader_1x01_P2.54mm_Vertical"
+		(locked yes)
 		(layer "F.Cu")
 		(at 50.16 31.62)
@@
 	)
 	(footprint "Connector_PinHeader_2.54mm:PinHeader_1x01_P2.54mm_Vertical"
+		(locked yes)
 		(layer "F.Cu")
-		(at 59.83 31.8)
+		(at 65.613333 31.62)
 		(descr "Through hole straight pin header, 1x01, 2.54mm pitch, single row")
 		(tags "Through hole pin header THT 1x01 2.54mm single row")
@@
 	(footprint "Resistor_THT:R_Axial_DIN0309_L9.0mm_D3.2mm_P15.24mm_Horizontal"
 		(layer "F.Cu")
-		(at 69.8 54.02 90)
+		(at 90.56 57.61 90)
 		(descr "Resistor, Axial_DIN0309 series, Axial, Horizontal, pin pitch=15.24mm, 0.5W = 1/2W, length*diameter=9*3.2mm^2, http://cdn-reichelt.de/documents/datenblatt/B400/1_4W%23YAG.pdf")
 		(tags "Resistor Axial_DIN0309 series Axial Horizontal pin pitch 15.24mm 0.5W = 1/2W length 9mm diameter 3.2mm")
 		(property "Reference" "R3"
-			(at 7.62 -2.72 90)
+			(at 17.25 -0.11 180)
 			(layer "F.SilkS")
 			(effects
@@
 	)
 	(footprint "Connector_PinHeader_2.54mm:PinHeader_1x01_P2.54mm_Vertical"
+		(locked yes)
 		(layer "F.Cu")
-		(at 79.66 31.87)
+		(at 96.52 31.62)
 		(descr "Through hole straight pin header, 1x01, 2.54mm pitch, single row")
 		(tags "Through hole pin header THT 1x01 2.54mm single row")

Commit message: Board outline
Other:
- board outline added: 68.7 x 62.7 mm
Changed lines of the file:
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@@
 		)
+	)
+	(gr_rect
+		(start 39.43 23.06)
+		(end 108.09 85.79)
+		(stroke
+			(width 0.05)
+			(type default)
+		)
+		(fill no)
+		(layer "Edge.Cuts")
 	)
 	(embedded_fonts no)

Commit message: Beautification
Other:
- board size 68.7 x 62.7 mm -> 68.7 x 67.5 mm
- board text added: "+5V"
- board text added: "-5V"
- board text added: "05-09-2026"
- board text added: "By - Mercy Presentia P (25BLC1150)"
- board text added: "Differential Amplifier - v1.0"
- board text added: "Op1"
- board text added: "Op2"
- board text added: "Vin1"
- board text added: "Vin2"
- board text added: "gnd"
Changed lines of the file:
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@@
 	)
 	(gr_rect
-		(start 39.43 23.06)
+		(start 39.43 18.33)
 		(end 108.09 85.79)
 		(stroke
@@
 		(layer "Edge.Cuts")
 	)
+	(gr_text "By - Mercy Presentia P (25BLC1150)"
+		(at 60.29 22.84 0)
+		(layer "F.SilkS")
+		(effects
+			(font
+				(size 1 1)
+				(thickness 0.1)
+			)
+			(justify left bottom)
+		)
+	)
+	(gr_text "Differential Amplifier - v1.0"
+		(at 63.73 20.63 0)
+		(layer "F.SilkS")
+		(effects
+			(font
+				(size 1 1)
+				(thickness 0.1)
+			)
+			(justify left bottom)
+		)
+	)
+	(gr_text "05-09-2026"
+		(at 96.98 20.46 0)
+		(layer "F.SilkS")
+		(effects
+			(font
+				(size 1 1)
+				(thickness 0.1)
+			)
+			(justify left bottom)
+		)
+	)
+	(gr_text "+5V"
+		(at 47.18 37.34 0)
+		(layer "F.SilkS")
+		(effects
+			(font
+				(size 2 2)
+				(thickness 0.2)
+			)
+			(justify left bottom)
+		)
+	)
+	(gr_text "Vin1"
+		(at 47.34 62.57 0)
+		(layer "F.SilkS")
+		(effects
+			(font
+				(size 2 2)
+				(thickness 0.2)
+			)
+			(justify left bottom)
+		)
+	)
+	(gr_text "gnd"
+		(at 47.34 83.21 0)
+		(layer "F.SilkS")
+		(effects
+			(font
+				(size 2 2)
+				(thickness 0.2)
+			)
+			(justify left bottom)
+		)
+	)
+	(gr_text "Op1"
+		(at 62.42 83.37 0)
+		(layer "F.SilkS")
+		(effects
+			(font
+				(size 2 2)
+				(thickness 0.2)
+			)
+			(justify left bottom)
+		)
+	)
+	(gr_text "gnd"
+		(at 63.07 36.93 0)
+		(layer "F.SilkS")
+		(effects
+			(font
+				(size 2 2)
+				(thickness 0.2)
+			)
+			(justify left bottom)
+		)
+	)
+	(gr_text "Vin2"
+		(at 68.56 62.57 0)
+		(layer "F.SilkS")
+		(effects
+			(font
+				(size 2 2)
+				(thickness 0.2)
+			)
+			(justify left bottom)
+		)
+	)
+	(gr_text "-5V"
+		(at 77.9 37.34 0)
+		(layer "F.SilkS")
+		(effects
+			(font
+				(size 2 2)
+				(thickness 0.2)
+			)
+			(justify left bottom)
+		)
+	)
+	(gr_text "gnd"
+		(at 78.47 83.21 0)
+		(layer "F.SilkS")
+		(effects
+			(font
+				(size 2 2)
+				(thickness 0.2)
+			)
+			(justify left bottom)
+		)
+	)
+	(gr_text "Op2"
+		(at 93.46 83.37 0)
+		(layer "F.SilkS")
+		(effects
+			(font
+				(size 2 2)
+				(thickness 0.2)
+			)
+			(justify left bottom)
+		)
+	)
+	(gr_text "gnd"
+		(at 93.95 36.68 0)
+		(layer "F.SilkS")
+		(effects
+			(font
+				(size 2 2)
+				(thickness 0.2)
+			)
+			(justify left bottom)
+		)
+	)
 	(embedded_fonts no)

Commit message: Routing done and ground filled
Routing:
- net Op2: track 0.00 -> 61.6 mm
- net Net-(Q1-S): track 0.00 -> 55.6 mm
- net Op1: track 0.00 -> 23.5 mm
- net Vdd: track 0.00 -> 22.4 mm
- net Vss: track 0.00 -> 14.7 mm
- net Vin2: track 0.00 -> 13.6 mm
- net Vin1: track 0.00 -> 12.9 mm
- added copper zone on F.Cu, net GND
Changed lines of the file:
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@@
 		)
 	)
-	(gr_text "gnd"
-		(at 78.47 83.21 0)
+	(gr_text "Op2"
+		(at 78.16 83.41 0)
 		(layer "F.SilkS")
 		(effects
@@
 		)
 	)
-	(gr_text "Op2"
-		(at 93.46 83.37 0)
+	(gr_text "gnd"
+		(at 93.85 83.12 0)
 		(layer "F.SilkS")
 		(effects
@@
 		)
 	)
+	(segment
+		(start 50.22 57.5)
+		(end 50.22 60.73)
+		(width 0.3)
+		(layer "F.Cu")
+		(net "Vin1")
+	)
+	(segment
+		(start 50.22 60.73)
+		(end 57.08 67.59)
+		(width 0.3)
+		(layer "F.Cu")
+		(net "Vin1")
+	)
+	(segment
+		(start 71.48 57.5)
+		(end 71.48 59.13)
+		(width 0.3)
+		(layer "F.Cu")
+		(net "Vin2")
+	)
+	(segment
+		(start 71.48 59.13)
+		(end 79.94 67.59)
+		(width 0.3)
+		(layer "F.Cu")
+		(net "Vin2")
+	)
+	(segment
+		(start 50.16 31.62)
+		(end 50.16 33.05)
+		(width 1)
+		(layer "F.Cu")
+		(net "Vdd")
+	)
+	(segment
+		(start 50.16 33.05)
+		(end 59.48 42.37)
+		(width 1)
+		(layer "F.Cu")
+		(net "Vdd")
+	)
+	(segment
+		(start 67.24 42.37)
+		(end 59.48 42.37)
+		(width 1)
+		(layer "F.Cu")
+		(net "Vdd")
+	)
+	(segment
+		(start 96 67.49)
+		(end 84.99 78.5)
+		(width 0.3)
+		(layer "F.Cu")
+		(net "Op2")
+	)
+	(segment
+		(start 96 55.88)
+		(end 96 67.49)
+		(width 0.3)
+		(layer "F.Cu")
+		(net "Op2")
+	)
+	(segment
+		(start 82.48 77.146)
+		(end 82.48 67.59)
+		(width 0.3)
+		(layer "F.Cu")
+		(net "Op2")
+	)
+	(segment
+		(start 81.126 78.5)
+		(end 82.48 77.146)
+		(width 0.3)
+		(layer "F.Cu")
+		(net "Op2")
+	)
+	(segment
+		(start 82.48 42.37)
+		(end 82.49 42.37)
+		(width 0.3)
+		(layer "F.Cu")
+		(net "Op2")
+	)
+	(segment
+		(start 84.99 78.5)
+		(end 81.126 78.5)
+		(width 0.3)
+		(layer "F.Cu")
+		(net "Op2")
+	)
+	(segment
+		(start 82.49 42.37)
+		(end 96 55.88)
+		(width 0.3)
+		(layer "F.Cu")
+		(net "Op2")
+	)
+	(segment
+		(start 59.62 72.447)
+		(end 59.62 67.59)
+		(width 0.3)
+		(layer "F.Cu")
+		(net "Op1")
+	)
+	(segment
+		(start 65.673 78.5)
+		(end 59.62 72.447)
+		(width 0.3)
+		(layer "F.Cu")
+		(net "Op1")
+	)
+	(segment
+		(start 59.48 67.45)
+		(end 59.62 67.59)
+		(width 0.3)
+		(layer "F.Cu")
+		(net "Op1")
+	)
+	(segment
+		(start 59.48 57.61)
+		(end 59.48 67.45)
+		(width 0.3)
+		(layer "F.Cu")
+		(net "Op1")
+	)
+	(segment
+		(start 62.16 67.59)
+		(end 65.89 63.86)
+		(width 0.3)
+		(layer "F.Cu")
+		(net "Net-(Q1-S)")
+	)
+	(segment
+		(start 70.81 50.54)
+		(end 79.72 50.54)
+		(width 0.3)
+		(layer "F.Cu")
+		(net "Net-(Q1-S)")
+	)
+	(segment
+		(start 86.83 57.61)
+		(end 90.56 57.61)
+		(width 0.3)
+		(layer "F.Cu")
+		(net "Net-(Q1-S)")
+	)
+	(segment
+		(start 90.56 57.61)
+		(end 90.56 62.05)
+		(width 0.3)
+		(layer "F.Cu")
+		(net "Net-(Q1-S)")
+	)
+	(segment
+		(start 65.89 55.46)
+		(end 70.81 50.54)
+		(width 0.3)
+		(layer "F.Cu")
+		(net "Net-(Q1-S)")
+	)
+	(segment
+		(start 65.89 63.86)
+		(end 65.89 55.46)
+		(width 0.3)
+		(layer "F.Cu")
+		(net "Net-(Q1-S)")
+	)
+	(segment
+		(start 90.56 62.05)
+		(end 85.02 67.59)
+		(width 0.3)
+		(layer "F.Cu")
+		(net "Net-(Q1-S)")
+	)
+	(segment
+		(start 79.72 50.54)
+		(end 79.74 50.52)
+		(width 0.3)
+		(layer "F.Cu")
+		(net "Net-(Q1-S)")
+	)
+	(segment
+		(start 79.74 50.52)
+		(end 86.83 57.61)
+		(width 0.3)
+		(layer "F.Cu")
+		(net "Net-(Q1-S)")
+	)
+	(segment
+		(start 90.56 41.113333)
+		(end 90.56 42.37)
+		(width 1)
+		(layer "F.Cu")
+		(net "Vss")
+	)
+	(segment
+		(start 81.066667 31.62)
+		(end 90.56 41.113333)
+		(width 1)
+		(layer "F.Cu")
+		(net "Vss")
+	)
+	(zone
+		(net "GND")
+		(layer "F.Cu")
+		(name "gnd")
+		(hatch edge 0.5)
+		(connect_pads
+			(clearance 0.5)
+		)
+		(min_thickness 0.25)
+		(fill yes
+			(thermal_gap 0.5)
+			(thermal_bridge_width 0.5)
+			(island_removal_mode 0)
+		)
+		(polygon
+			(pts
+				(xy 36.36 15.53) (xy 36.6 91.47) (xy 113.52 91.59) (xy 113.52 15.53) (xy 36.48 15.65)
+			)
+		)
+	)
